File: Schematic/Thermostat/Thermostat.kicad_sch (KiCad schematic)
At the start: 27 parts, among them J1 Heater, J2 230VAC IN, U1 TS321ILT

Commit message: Rearranged schematic, added copy ring
Other:
- company: (none) -> Retronics - Bjørner Sandom
- title: (none) -> PlantShelf Thermostat
Changed lines of the file:
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@@
 	(generator_version "8.0")
 	(paper "A4")
+	(title_block
+		(title "PlantShelf Thermostat")
+		(date "2025-04-06")
+		(company "Retronics - Bjørner Sandom")
+	)
 	(junction
 		(at 146.05 55.88)
